Commit message: Revised URDF files (#228)

File: dsr_description2/urdf/a0509.blue.urdf (robot description, URDF)
Before this commit: robot a0509, 8 links, 7 joints
Joints:
- joint joint_1: origin xyz=0 0 0.1555 rpy=0 0 0 -> xyz=0 0 0.1560 rpy=0 0 0

File: dsr_description2/urdf/a0509.urdf (robot description, URDF)
Before this commit: robot a0509, 8 links, 7 joints
Joints:
- joint joint_1: origin xyz=0 0 0.1555 rpy=0 0 0 -> xyz=0 0 0.1560 rpy=0 0 0

File: dsr_description2/urdf/a0509.white.urdf (robot description, URDF)
Before this commit: robot a0509, 8 links, 7 joints
Joints:
- joint joint_1: origin xyz=0 0 0.1555 rpy=0 0 0 -> xyz=0 0 0.1560 rpy=0 0 0

File: dsr_description2/urdf/m0609.blue.urdf (robot description, URDF)
Before this commit: robot m0609, 8 links, 7 joints
Joints:
- joint joint_1: origin xyz=0 0 0.1525 rpy=0 0 0 -> xyz=0 0 0.1345 rpy=0 0 0

File: dsr_description2/urdf/m0609.urdf (robot description, URDF)
Before this commit: robot m0609, 9 links, 8 joints
Joints:
- joint joint_1: origin xyz=0 0 0.1 rpy=0 0 0 -> xyz=0 0 0.1345 rpy=0 0 0

File: dsr_description2/urdf/m0609.white.urdf (robot description, URDF)
Before this commit: robot m0609, 8 links, 7 joints
Joints:
- joint joint_1: origin xyz=0 0 0.1525 rpy=0 0 0 -> xyz=0 0 0.1345 rpy=0 0 0

File: dsr_description2/urdf/m0617.blue.urdf (robot description, URDF)
Before this commit: robot m0617, 8 links, 7 joints
Joints:
- joint joint_1: origin xyz=0 0 0.1525 rpy=0 0 0 -> xyz=0 0 0.1530 rpy=0 0 0

File: dsr_description2/urdf/m0617.urdf (robot description, URDF)
Before this commit: robot m0617, 8 links, 7 joints
Joints:
- joint joint_1: origin xyz=0 0 0.1525 rpy=0 0 0 -> xyz=0 0 0.1530 rpy=0 0 0

File: dsr_description2/urdf/m0617.white.urdf (robot description, URDF)
Before this commit: robot m0617, 8 links, 7 joints
Joints:
- joint joint_1: origin xyz=0 0 0.1525 rpy=0 0 0 -> xyz=0 0 0.1530 rpy=0 0 0

File: dsr_description2/urdf/m1509.blue.urdf (robot description, URDF)
Before this commit: robot m1509, 8 links, 7 joints
Joints:
- joint joint_1: origin xyz=0 0 0.1525 rpy=0 0 0 -> xyz=0 0 0.1530 rpy=0 0 0

File: dsr_description2/urdf/m1509.urdf (robot description, URDF)
Before this commit: robot m1509, 8 links, 7 joints
Joints:
- joint joint_1: origin xyz=0 0 0.1525 rpy=0 0 0 -> xyz=0 0 0.1530 rpy=0 0 0

File: dsr_description2/urdf/m1509.white.urdf (robot description, URDF)
Before this commit: robot m1509, 8 links, 7 joints
Joints:
- joint joint_1: origin xyz=0 0 0.1525 rpy=0 0 0 -> xyz=0 0 0.1530 rpy=0 0 0
