Commit message: fix: gazebo failing to run some robots

File: dsr_description2/xacro/a0509.urdf.xacro (robot description, xacro)
@@ -25,9 +25,9 @@
     <child  link="base_link"/>
   </joint>
-  <xacro:if value="${gz == 'true'}">
+  <xacro:if value="${gz}">
     <xacro:include filename="$(find dsr_description2)/ros2_control/a0509.gz_ros2_control.xacro"/>
     <xacro:a0509_gz_ros2_control namespace="$(arg namespace)"/>
   </xacro:if>
-  <xacro:unless value="${gz == 'true'}">
+  <xacro:unless value="${gz}">
     <xacro:include filename="$(find dsr_description2)/ros2_control/a0509.ros2_control.xacro"/>
     <xacro:a0509_ros2_control name="a0509"/>

File: dsr_description2/xacro/a0912.urdf.xacro (robot description, xacro)
@@ -25,9 +25,9 @@
     <child  link="base_link"/>
   </joint>
-  <xacro:if value="${gz == 'true'}">
+  <xacro:if value="${gz}">
     <xacro:include filename="$(find dsr_description2)/ros2_control/a0912.gz_ros2_control.xacro"/>
     <xacro:a0912_gz_ros2_control namespace="$(arg namespace)"/>
   </xacro:if>
-  <xacro:unless value="${gz == 'true'}">
+  <xacro:unless value="${gz}">
     <xacro:include filename="$(find dsr_description2)/ros2_control/a0912.ros2_control.xacro"/>
     <xacro:a0912_ros2_control name="a0912"/>

File: dsr_description2/xacro/e0509.urdf.xacro (robot description, xacro)
@@ -25,9 +25,9 @@
     <child  link="base_link"/>
   </joint>
-  <xacro:if value="${gz == 'true'}">
+  <xacro:if value="${gz}">
     <xacro:include filename="$(find dsr_description2)/ros2_control/e0509.gz_ros2_control.xacro"/>
     <xacro:e0509_gz_ros2_control namespace="$(arg namespace)"/>
   </xacro:if>
-  <xacro:unless value="${gz == 'true'}">
+  <xacro:unless value="${gz}">
     <xacro:include filename="$(find dsr_description2)/ros2_control/e0509.ros2_control.xacro"/>
     <xacro:e0509_ros2_control name="e0509"/>

File: dsr_description2/xacro/h2017.urdf.xacro (robot description, xacro)
@@ -25,9 +25,9 @@
     <child  link="base_link"/>
   </joint>
-  <xacro:if value="${gz == 'true'}">
+  <xacro:if value="${gz}">
     <xacro:include filename="$(find dsr_description2)/ros2_control/h2017.gz_ros2_control.xacro"/>
     <xacro:h2017_gz_ros2_control namespace="$(arg namespace)"/>
   </xacro:if>
-  <xacro:unless value="${gz == 'true'}">
+  <xacro:unless value="${gz}">
     <xacro:include filename="$(find dsr_description2)/ros2_control/h2017.ros2_control.xacro"/>
     <xacro:h2017_ros2_control name="h2017"/>

File: dsr_description2/xacro/h2515.urdf.xacro (robot description, xacro)
@@ -25,9 +25,9 @@
     <child  link="base_link"/>
   </joint>
-  <xacro:if value="${gz == 'true'}">
+  <xacro:if value="${gz}">
     <xacro:include filename="$(find dsr_description2)/ros2_control/h2515.gz_ros2_control.xacro"/>
     <xacro:h2515_gz_ros2_control namespace="$(arg namespace)"/>
   </xacro:if>
-  <xacro:unless value="${gz == 'true'}">
+  <xacro:unless value="${gz}">
     <xacro:include filename="$(find dsr_description2)/ros2_control/h2515.ros2_control.xacro"/>
     <xacro:h2515_ros2_control name="h2515"/>

File: dsr_description2/xacro/m0609.urdf.xacro (robot description, xacro)
@@ -25,10 +25,10 @@
     <child  link="base_link"/>
   </joint>
-  <xacro:if value="${gz == 'true'}">
+  <xacro:if value="${gz}">
     <xacro:include filename="$(find dsr_description2)/ros2_control/m0609.gz_ros2_control.xacro"/>
     <xacro:m0609_gz_ros2_control namespace="$(arg namespace)"/>
   </xacro:if>
-  <xacro:unless value="${gz == 'true'}">
-    <xacro:include filename="$(find dsr_description2)/ros2_control/mm0609.ros2_control.xacro"/>
+  <xacro:unless value="${gz}">
+    <xacro:include filename="$(find dsr_description2)/ros2_control/m0609.ros2_control.xacro"/>
     <xacro:m0609_ros2_control name="m0609"/>
   </xacro:unless>

File: dsr_description2/xacro/m0617.urdf.xacro (robot description, xacro)
@@ -25,9 +25,9 @@
     <child  link="base_link"/>
   </joint>
-  <xacro:if value="${gz == 'true'}">
+  <xacro:if value="${gz}">
     <xacro:include filename="$(find dsr_description2)/ros2_control/m0617.gz_ros2_control.xacro"/>
     <xacro:m0617_gz_ros2_control namespace="$(arg namespace)"/>
   </xacro:if>
-  <xacro:unless value="${gz == 'true'}">
+  <xacro:unless value="${gz}">
     <xacro:include filename="$(find dsr_description2)/ros2_control/m0617.ros2_control.xacro"/>
     <xacro:m0617_ros2_control name="m0617"/>

File: dsr_description2/xacro/m1509.urdf.xacro (robot description, xacro)
@@ -25,9 +25,9 @@
     <child  link="base_link"/>
   </joint>
-  <xacro:if value="${gz == 'true'}">
+  <xacro:if value="${gz}">
     <xacro:include filename="$(find dsr_description2)/ros2_control/m1509.gz_ros2_control.xacro"/>
     <xacro:m1509_gz_ros2_control namespace="$(arg namespace)"/>
   </xacro:if>
-  <xacro:unless value="${gz == 'true'}">
+  <xacro:unless value="${gz}">
     <xacro:include filename="$(find dsr_description2)/ros2_control/m1509.ros2_control.xacro"/>
     <xacro:m1509_ros2_control name="m1509"/>

File: dsr_description2/xacro/macro.p3020.white.xacro (robot description, xacro)
@@ -11,6 +11,6 @@
                 <mass value="9.55"/>
                 <origin xyz="6e-06   -0.007232     0.10749"/>
-                <inertia ixx="0.11196" ixy="1.4011e-05" ixz="-0.0049962" iyy="0.0065009" iyz="-0.004993"
-                        izz="0.0056525"/>
+                <!-- TODO: add real inertial values -->
+                <inertia ixx="1" ixy="0" ixz="0" iyy="1" iyz="0" izz="1"/>
             </inertial>
             <visual>

File: dsr_description2/xacro/p3020.urdf.xacro (robot description, xacro)
@@ -25,9 +25,9 @@
     <child  link="base_link"/>
   </joint>
-  <xacro:if value="${gz == 'true'}">
+  <xacro:if value="${gz}">
     <xacro:include filename="$(find dsr_description2)/ros2_control/p3020.gz_ros2_control.xacro"/>
     <xacro:p3020_gz_ros2_control namespace="$(arg namespace)"/>
   </xacro:if>
-  <xacro:unless value="${gz == 'true'}">
+  <xacro:unless value="${gz}">
     <xacro:include filename="$(find dsr_description2)/ros2_control/p3020.ros2_control.xacro"/>
     <xacro:p3020_ros2_control name="p3020"/>
