Commit message: Adding the nginx stackbot config file (#307)

File: dsr_description2/ros2_control/p3020.gz_ros2_control.xacro (robot description, xacro)
@@ -14,5 +14,5 @@
   mobile:=none
   use_gazebo:=false
-  update_rate
+  update_rate:=100
   ">
   <xacro:property name="double_pi" value="${2.0 * pi}"/>

File: dsr_description2/ros2_control/p3020.ros2_control.xacro (robot description, xacro)
@@ -8,5 +8,5 @@
   mode:=real
   model:=p3020
-  update_rate
+  update_rate:=100
   ">
     <xacro:property name="double_pi" value="${2.0 * pi}"/>

File: dsr_description2/xacro/p3020.urdf.xacro (robot description, xacro)
@@ -9,4 +9,5 @@
   <xacro:arg name="mode" default=""/>
   <xacro:arg name="model" default=""/>
+  <xacro:arg name="update_rate" default=""/>
   <!-- gripper control argument -->
   <xacro:arg name="gripper"              default="none"/>         <!-- none | robotique -->
@@ -20,4 +21,5 @@
   <xacro:property name="mode" value="$(arg mode)"/>
   <xacro:property name="model" value="$(arg model)"/>
+  <xacro:property name="update_rate" value="$(arg update_rate)"/>
   <xacro:property name="cr" value="$(arg color)"/>
   <xacro:property name="gr" value="$(arg gripper)"/>
@@ -48,4 +50,5 @@
       mode="${mode}"
       model="${model}"
+      update_rate="${update_rate}"
     />
   </xacro:unless>
