Commit message: Update mobile manipulator

File: dsr_description2/config/macro.materials.xacro (robot description, xacro)
@@ -20,4 +20,10 @@
 			<color rgba="0 0 0.15 1" />
 		</material>
+		<material name="grey">
+			<color rgba="0.5 0.5 0.5 1.0" />
+		</material>
+		<material name="Boxer_DarkGrey">
+			<color rgba="0.3 0.3 0.3 1.0" />
+		</material>
 	</xacro:macro>
 </robot>
